File: previous version archive/LMP848x Breakout v1.3.brd (EAGLE design)
At the start: 47.9 x 43.2 mm, 32 parts, among them X1 MINI-USB-UX60-MB-5ST

Commit message: v1.4 commit
Parts:
- moved C1 0.51 mm to (28.4, 27.9)
- moved C2 0.51 mm to (28.4, 17.8)
- moved X1 0.27 mm to (34.5, 6.85)
- renumbered LMP848X to LMP8481
Connections:
- net N$5: now also SV1.3; no longer SV1.2
- net N$6: now also SV1.2
- net VDIV: now also SV1.4; no longer SV1.3
Routing:
- net N$6: track 14.7 -> 36.9 mm
- net N$5: track 6.56 -> 7.78 mm
- net VDIV: track 35.5 -> 36.5 mm
